File: cheapsplit.sch (KiCad schematic (older format))
At the start: 51 parts, among them J1 AudioJack4, SW1 SW_Push, SW10 SW_Push, SW11 SW_Push, SW12 SW_Push, SW13 SW_Push, SW14 SW_Push, SW15 SW_Push, SW16 SW_Push, SW17 SW_Push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

Commit message: Finished pcb
Parts:
- JP1, JP2, JP3: footprint Connector_PinHeader_1.00mm:PinHeader_1x03_P1.00mm_Vertical -> Connector_PinHeader_1.27mm:PinHeader_1x03_P1.27mm_Vertical
Connections:
- net col0: now also B1.10 (7)
- net col1: now also B1.9 (*6)
- net col2: now also B1.8 (*5)
- net col3: now also B1.7 (4)
- net col4: now also B1.15 (12(MISO))
- net row0: now also B1.5 (2)
- net row1: now also B1.6 (*3)
- net row2: now also B1.11 (8)
- net row3: now also B1.12 (*9)
Other:
- moved on the sheet: JP1
Changed lines of the file:
@@
 F 0 "JP2" H 9050 2681 50  0000 C CNN
 F 1 "Jumper_3_Open" H 9050 2772 50  0000 C CNN
-F 2 "Connector_PinHeader_1.00mm:PinHeader_1x03_P1.00mm_Vertical" H 9050 2550 50  0001 C CNN
+F 2 "Connector_PinHeader_1.27mm:PinHeader_1x03_P1.27mm_Vertical" H 9050 2550 50  0001 C CNN
 F 3 "~" H 9050 2550 50  0001 C CNN
 	1    9050 2550
@@
 F 0 "JP3" H 9050 5024 50  0000 C CNN
 F 1 "Jumper_3_Open" H 9050 4933 50  0000 C CNN
-F 2 "Connector_PinHeader_1.00mm:PinHeader_1x03_P1.00mm_Vertical" H 9050 4800 50  0001 C CNN
+F 2 "Connector_PinHeader_1.27mm:PinHeader_1x03_P1.27mm_Vertical" H 9050 4800 50  0001 C CNN
 F 3 "~" H 9050 4800 50  0001 C CNN
 	1    9050 4800
@@
 $EndComp
 Wire Wire Line
-	8600 3300 8350 3300
+	8600 3300 8300 3300
 Wire Wire Line
-	8350 3300 8350 2550
+	8300 3300 8300 2550
 Wire Wire Line
-	8350 2550 8800 2550
+	8300 2550 8800 2550
 Wire Wire Line
-	9500 3300 9750 3300
+	9500 3300 9800 3300
 Wire Wire Line
-	9750 3300 9750 2550
+	9800 3300 9800 2550
 Wire Wire Line
-	9750 2550 9300 2550
+	9800 2550 9300 2550
 Text GLabel 9100 2350 2    50   Input ~ 0
 TX
@@
 NoConn ~ 6050 7300
 Wire Wire Line
-	9500 3600 9750 3600
+	9500 3600 9800 3600
 Wire Wire Line
-	9750 3600 9750 4800
+	9800 3600 9800 4800
 Wire Wire Line
-	9750 4800 9300 4800
+	9800 4800 9300 4800
 Wire Wire Line
-	8600 3600 8350 3600
+	8600 3600 8300 3600
 Wire Wire Line
-	8350 3600 8350 4800
+	8300 3600 8300 4800
 Wire Wire Line
-	8350 4800 8800 4800
+	8300 4800 8800 4800
 $Comp
 L power:+5V #PWR0103
@@
 L Jumper:Jumper_3_Open JP1
 U 1 1 6109A03A
-P 7550 3450
-F 0 "JP1" V 7504 3537 50  0000 L CNN
-F 1 "Jumper_3_Open" V 7595 3537 50  0000 L CNN
-F 2 "Connector_PinHeader_1.00mm:PinHeader_1x03_P1.00mm_Vertical" H 7550 3450 50  0001 C CNN
-F 3 "~" H 7550 3450 50  0001 C CNN
-	1    7550 3450
+P 7500 3450
+F 0 "JP1" V 7454 3537 50  0000 L CNN
+F 1 "Jumper_3_Open" V 7545 3537 50  0000 L CNN
+F 2 "Connector_PinHeader_1.27mm:PinHeader_1x03_P1.27mm_Vertical" H 7500 3450 50  0001 C CNN
+F 3 "~" H 7500 3450 50  0001 C CNN
+	1    7500 3450
 	0    1    1    0
 $EndComp
 Wire Wire Line
-	8600 3500 8250 3500
+	8600 3500 8200 3500
 Wire Wire Line
-	8250 3500 8250 3800
+	8200 3500 8200 3800
 Wire Wire Line
-	8250 3800 7550 3800
+	8200 3800 7500 3800
 Wire Wire Line
-	7550 3800 7550 3700
+	7500 3800 7500 3700
 Wire Wire Line
-	8600 3400 8250 3400
+	8600 3400 8200 3400
 Wire Wire Line
-	8250 3400 8250 3100
+	8200 3400 8200 3100
 Wire Wire Line
-	8250 3100 7550 3100
+	8200 3100 7500 3100
 Wire Wire Line
-	7550 3100 7550 3200
+	7500 3100 7500 3200
 $Comp
 L power:GND #PWR0104
@@
 	7200 3600 7200 3450
 Wire Wire Line
-	7200 3450 7400 3450
+	7200 3450 7350 3450
 NoConn ~ 9500 3500
 NoConn ~ 9500 3400
@@
 	1    0    0    -1
 $EndComp
+Text GLabel 8600 3700 0    50   Input ~ 0
+row0
+Text GLabel 8600 3800 0    50   Input ~ 0
+row1
+Text GLabel 8600 4300 0    50   Input ~ 0
+row2
+Text GLabel 8600 4400 0    50   Input ~ 0
+row3
+Text GLabel 8600 4200 0    50   Input ~ 0
+col0
+Text GLabel 8600 4100 0    50   Input ~ 0
+col1
+Text GLabel 8600 4000 0    50   Input ~ 0
+col2
+Text GLabel 8600 3900 0    50   Input ~ 0
+col3
+Text GLabel 9500 4200 2    50   Input ~ 0
+col4
 $EndSCHEMATC
